File: Lifedatalink_v1_revA.sch (KiCad schematic (older format))
At the start: 60 parts, among them J1 DX07S024XJ1R1100, J2 BATTERY CONNECTOR, J3 DF17(4.0)-30DS-0.5V(57), J4 503480-0600, Q1 DMG2301L, U1 BL654, U2 LP5907MFX-3_3_NOPB, U3 ADS1292R, U4 MCP73831-2-OT, U5 TMP117NAIYBGR, U6 MAX30102, U7 LP5907MFX-1.8, Y1 Crystal

Commit message: Hexagonal PCB placed
Parts:
- removed J3: DF17(4.0)-30DS-0.5V(57), HRS_DF17(4.0)-30DS-0:HRS_DF17(4.0)-30DS-0.5V(57), symbol DF17_4.0_-30DS-0.5V_57_:DF17(4.0)-30DS-0.5V(57)
- added J10, J5, J6, J7, J8, J9: 503480-0400, 503480-0400:MOLEX_503480-0400, symbol 503480-0400:503480-0400
- added J11, J12: 5034801000, MOLEX_503480-0600:MOLEX_5034801000, symbol 503480-1000:5034801000
- added J13, J14, J15, J16: 503480-0600, MOLEX_503480-0600:MOLEX_503480-0600, symbol 503480-0600:503480-0600
- added J3: Conn_02x10_Odd_Even, DF23:DF23C-20DS-0.5V(51), symbol Connector_Generic:Conn_02x10_Odd_Even
- D3: footprint digikey-footprints:SOD-123 -> Diode_SMD:D_SOD-123
- J2: footprint Connector_JST:JST_PH_S2B-PH-SM4-TB_1x02-1MP_P2.00mm_Horizontal -> Connector_PinHeader_2.00mm:PinHeader_1x02_P2.00mm_Vertical
- Q1: footprint digikey-footprints:SOT-23-3 -> Package_TO_SOT_SMD:SOT-23
Connections:
- net labels added: TMP_ADD0
- wire segments 273 -> 307
Other:
- moved on the sheet: C24, U5, U6

Commit message: Added ECG snaps, microphones and other 3D models.
Parts:
- removed J11, J12: 5034801000, MOLEX_503480-0600:MOLEX_5034801000, symbol 503480-1000:5034801000
- removed J4: 503480-0600, MOLEX_503480-0600:MOLEX_503480-0600, symbol 503480-0600:503480-0600
- added C27: 100nF, Capacitor_SMD:C_0402_1005Metric, symbol Device:C
- added C28: 10uF, Capacitor_SMD:C_0402_1005Metric, symbol Device:C
- added C29, C30: 0.1uF, Capacitor_SMD:C_0402_1005Metric, symbol Device:C
- added J11, J12: 5034801400, MOLEX_503480-0600:5034801400, symbol Connector_Generic_Shielded:Conn_01x14_Shielded
- added J17, J18, J19, J20: 503480-0600, MOLEX_503480-0600:MOLEX_503480-0600, symbol 503480-0600:503480-0600
- added J4: Conn_01x06, Pads_1.27mm:1.27mm_pads_01x06, symbol Connector_Generic:Conn_01x06
- added MIC1, MIC2: ICS-43434, digikey-footprints:SPH0645LM4H-B, symbol dk_Microphones:SPH0645LM4H-B
- added R17: 200K, Resistor_SMD:R_0402_1005Metric, symbol Device:R
- added R20, R21: 4.7K, Resistor_SMD:R_0402_1005Metric, symbol Device:R
- added R22: 100K, Resistor_SMD:R_0402_1005Metric, symbol Device:R
- added U8: IIS2DLPCTR, Package_LGA:LGA-12_2x2mm_P0.5mm, symbol IIS2DLPCTR:IIS2DLPCTR
- added U9: PCA9306, Package_SON:X2SON-8_1.4x1mm_P0.35mm, symbol Interface:PCA9306
- D3: footprint Diode_SMD:D_SOD-123 -> Diode_SMD:D_SOD-123F
Connections:
- net labels added: ACCEL_INT1, ACCEL_INT2, BL654_I2C_SCL_HV, BL654_I2C_SCL_LV, BL654_I2C_SDA_HV, BL654_I2C_SDA_LV, BL654_I2S_SCK, BL654_I2S_SD, BL654_I2S_WS
- net labels removed: BL654_I2C_SCL, BL654_I2C_SDA
- wire segments 307 -> 388
Other:
- note added: "1.8V LDO"
- note added: "3.3V LDO"
- note added: "I2C LEVEL SHIFTER"
- note added: "LEFT"
- note added: "RIGHT"
- moved on the sheet: C24, C25, C26, C3, C4, D3, J10, J13, J14, J15, J16, J5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

Commit message: Fixed LED and added JST connector to battery plus more 3D models
Parts:
- removed D2: LTST-C155KGJRKT, SeeedOPL-LED:LED_Cree-PLCC4_3.2x2.8mm_CCW_jose, symbol Device:LED_Dual_AACC
- removed R1, R2: 470, Resistor_SMD:R_0402_1005Metric, symbol Device:R
- added D?: WS2812B, APA-102-2020-256-8:LED_WS2812-2020, symbol LED:WS2812B
- added F1: 0603L075SLYR, Fuse:Fuse_0603_1608Metric, symbol Device:Fuse
- J2: footprint Connector_PinHeader_2.00mm:PinHeader_1x02_P2.00mm_Vertical -> Connector_JST:JST_SH_BM02B-SRSS-TB_1x02-1MP_P1.00mm_Vertical
Connections:
- net labels added: MCP73831_STAT, VIN, WS2812_DATA
- wire segments 388 -> 376
Other:
- moved on the sheet: C4, U2
Changed lines of the file:
@@
 $EndComp
 $Comp
-L Device:R R1
-U 1 1 5E7F6934
-P 6400 2200
-F 0 "R1" V 6480 2200 50  0000 C CNN
-F 1 "470" V 6400 2200 50  0000 C CNN
-F 2 "Resistor_SMD:R_0402_1005Metric" V 6330 2200 50  0001 C CNN
-F 3 "~" H 6400 2200 50  0001 C CNN
-	1    6400 2200
-	0    1    1    0
-$EndComp
-$Comp
-L Device:R R2
-U 1 1 5E7F77E5
-P 6400 2400
-F 0 "R2" V 6480 2400 50  0000 C CNN
-F 1 "470" V 6400 2400 50  0000 C CNN
-F 2 "Resistor_SMD:R_0402_1005Metric" V 6330 2400 50  0001 C CNN
-F 3 "~" H 6400 2400 50  0001 C CNN
-	1    6400 2400
-	0    1    1    0
-$EndComp
-$Comp
-L Device:LED_Dual_AACC D2
-U 1 1 5E7F9C1C
-P 7700 2300
-F 0 "D2" H 7700 2525 50  0000 C CNN
-F 1 "LTST-C155KGJRKT" H 7700 2050 50  0000 C CNN
-F 2 "SeeedOPL-LED:LED_Cree-PLCC4_3.2x2.8mm_CCW_jose" H 7730 2300 50  0001 C CNN
-F 3 "~" H 7730 2300 50  0001 C CNN
-F 4 "LTST-C155KGJRKT" H 7700 2300 50  0001 C CNN "MPN"
-	1    7700 2300
-	-1   0    0    1
-$EndComp
-$Comp
 L Device:R R3
 U 1 1 5E80F2F0
@@
 $EndComp
 Wire Wire Line
-	6050 2200 6150 2200
-Wire Wire Line
-	6150 2200 6150 2400
-Wire Wire Line
-	6150 2400 6250 2400
-Connection ~ 6150 2200
-Wire Wire Line
-	6150 2200 6250 2200
-Wire Wire Line
-	6550 2400 6700 2400
-Wire Wire Line
-	6700 2400 6700 2750
-Wire Wire Line
-	8150 2750 8150 2400
-Wire Wire Line
-	8150 2400 8000 2400
-$Comp
-L power:GND #PWR023
-U 1 1 5E7F083E
-P 7150 2500
-F 0 "#PWR023" H 7150 2250 50  0001 C CNN
-F 1 "GND" H 7150 2350 50  0000 C CNN
-F 2 "" H 7150 2500 50  0001 C CNN
-F 3 "" H 7150 2500 50  0001 C CNN
-	1    7150 2500
-	1    0    0    -1
-$EndComp
-Wire Wire Line
-	7150 2500 7150 2400
-Wire Wire Line
-	7150 2400 7400 2400
-$Comp
-L power:+5V #PWR022
-U 1 1 5E7F58DA
-P 8150 1900
-F 0 "#PWR022" H 8150 1750 50  0001 C CNN
-F 1 "+5V" H 8150 2040 50  0000 C CNN
-F 2 "" H 8150 1900 50  0001 C CNN
-F 3 "" H 8150 1900 50  0001 C CNN
-	1    8150 1900
-	1    0    0    -1
-$EndComp
-Wire Wire Line
-	8000 2200 8150 2200
-Wire Wire Line
-	8150 2200 8150 1900
-Wire Wire Line
 	4950 2350 4950 2200
 Wire Wire Line
@@
 F 0 "J2" H 7600 1650 50  0000 C CNN
 F 1 "BATTERY CONNECTOR" H 7600 1350 50  0000 C CNN
-F 2 "Connector_PinHeader_2.00mm:PinHeader_1x02_P2.00mm_Vertical" H 7600 1550 50  0001 C CNN
+F 2 "Connector_JST:JST_SH_BM02B-SRSS-TB_1x02-1MP_P1.00mm_Vertical" H 7600 1550 50  0001 C CNN
 F 3 "~" H 7600 1550 50  0001 C CNN
 	1    7600 1550
@@
 Connection ~ 5600 8300
 Wire Wire Line
-	6550 2200 7400 2200
-Wire Wire Line
-	6700 2750 8150 2750
-Wire Wire Line
 	7100 1550 7400 1550
 Wire Wire Line
@@
 BL654_SWDCLK
 $Comp
-L power:+3.3V #PWR050
-U 1 1 5ED512AD
-P 17150 6050
-F 0 "#PWR050" H 17150 5900 50  0001 C CNN
-F 1 "+3.3V" H 17150 6190 50  0000 C CNN
-F 2 "" H 17150 6050 50  0001 C CNN
-F 3 "" H 17150 6050 50  0001 C CNN
-	1    17150 6050
-	1    0    0    -1
-$EndComp
-$Comp
 L power:GND #PWR051
 U 1 1 5ED51BC6
@@
 	1    0    0    -1
 $EndComp
-Text Notes 10300 1600 0    50   ~ 0
+Text Notes 10850 1600 0    50   ~ 0
 3.3V LDO
 $Comp
 L power:+3.3V #PWR06
 U 1 1 5E7FBE04
-P 10950 1750
-F 0 "#PWR06" H 10950 1600 50  0001 C CNN
-F 1 "+3.3V" H 10950 1890 50  0000 C CNN
-F 2 "" H 10950 1750 50  0001 C CNN
-F 3 "" H 10950 1750 50  0001 C CNN
-	1    10950 1750
+P 11500 1750
+F 0 "#PWR06" H 11500 1600 50  0001 C CNN
+F 1 "+3.3V" H 11500 1890 50  0000 C CNN
+F 2 "" H 11500 1750 50  0001 C CNN
+F 3 "" H 11500 1750 50  0001 C CNN
+	1    11500 1750
 	1    0    0    -1
 $EndComp
@@
 	9550 2150 9700 2150
 Wire Wire Line
-	10300 2450 10300 2700
+	10850 2450 10850 2700
 $Comp
 L power:GND #PWR010
 U 1 1 5E8006E0
-P 10300 2700
-F 0 "#PWR010" H 10300 2450 50  0001 C CNN
-F 1 "GND" H 10300 2550 50  0000 C CNN
-F 2 "" H 10300 2700 50  0001 C CNN
-F 3 "" H 10300 2700 50  0001 C CNN
-	1    10300 2700
+P 10850 2700
+F 0 "#PWR010" H 10850 2450 50  0001 C CNN
+F 1 "GND" H 10850 2550 50  0000 C CNN
+F 2 "" H 10850 2700 50  0001 C CNN
+F 3 "" H 10850 2700 50  0001 C CNN
+	1    10850 2700
 	1    0    0    -1
 $EndComp
 Wire Wire Line
-	10950 2600 10950 2700
-Connection ~ 10950 2150
+	11500 2600 11500 2700
+Connection ~ 11500 2150
 Wire Wire Line
-	10950 2300 10950 2150
+	11500 2300 11500 2150
 Wire Wire Line
-	10950 2150 10950 1750
+	11500 2150 11500 1750
 Wire Wire Line
-	10600 2150 10950 2150
+	11150 2150 11500 2150
 Wire Wire Line
-	9900 2150 10000 2150
-Connection ~ 9900 2150
+	10450 2150 10550 2150
 Wire Wire Line
-	9900 2250 9900 2150
+	10450 2250 10450 2150
 Wire Wire Line
-	10000 2250 9900 2250
+	10550 2250 10450 2250
 Wire Wire Line
 	9700 2150 9700 2300
 Wire Wire Line
-	9700 2150 9900 2150
-Wire Wire Line
 	9700 2600 9700 2700
 $Comp
 L power:GND #PWR011
 U 1 1 5E7FCAC1
-P 10950 2700
-F 0 "#PWR011" H 10950 2450 50  0001 C CNN
-F 1 "GND" H 10950 2550 50  0000 C CNN
-F 2 "" H 10950 2700 50  0001 C CNN
-F 3 "" H 10950 2700 50  0001 C CNN
-	1    10950 2700
+P 11500 2700
+F 0 "#PWR011" H 11500 2450 50  0001 C CNN
+F 1 "GND" H 11500 2550 50  0000 C CNN
+F 2 "" H 11500 2700 50  0001 C CNN
+F 3 "" H 11500 2700 50  0001 C CNN
+	1    11500 2700
 	1    0    0    -1
 $EndComp
@@
 L Device:C C4
 U 1 1 5E7FAF22
-P 10950 2450
-F 0 "C4" H 10975 2550 50  0000 L CNN
-F 1 "1uF" H 10975 2350 50  0000 L CNN
-F 2 "Capacitor_SMD:C_0402_1005Metric" H 10988 2300 50  0001 C CNN
-F 3 "~" H 10950 2450 50  0001 C CNN
-	1    10950 2450
+P 11500 2450
+F 0 "C4" H 11525 2550 50  0000 L CNN
+F 1 "1uF" H 11525 2350 50  0000 L CNN
+F 2 "Capacitor_SMD:C_0402_1005Metric" H 11538 2300 50  0001 C CNN
+F 3 "~" H 11500 2450 50  0001 C CNN
+	1    11500 2450
 	-1   0    0    1
 $EndComp
@@
 L dk_PMIC-Voltage-Regulators-Linear:LP5907MFX-3_3_NOPB U2
 U 1 1 5E7F886D
-P 10300 2350
-F 0 "U2" H 10300 2700 60  0000 C CNN
-F 1 "LP5907MFX-3_3_NOPB" H 10300 2800 60  0000 C CNN
-F 2 "Package_TO_SOT_SMD:SOT-23-5" H 10500 2550 60  0001 L CNN
-F 3 "http://www.ti.com/general/docs/suppproductinfo.tsp?distId=10&gotoUrl=http%3A%2F%2Fwww.ti.com%2Flit%2Fgpn%2Flp5907" H 10500 2650 60  0001 L CNN
-F 4 "296-38557-1-ND" H 10500 2750 60  0001 L CNN "Digi-Key_PN"
-F 5 "LP5907MFX-3.3/NOPB" H 10500 2850 60  0001 L CNN "MPN"
-F 6 "Integrated Circuits (ICs)" H 10500 2950 60  0001 L CNN "Category"
-F 7 "PMIC - Voltage Regulators - Linear" H 10500 3050 60  0001 L CNN "Family"
-F 8 "http://www.ti.com/general/docs/suppproductinfo.tsp?distId=10&gotoUrl=http%3A%2F%2Fwww.ti.com%2Flit%2Fgpn%2Flp5907" H 10500 3150 60  0001 L CNN "DK_Datasheet_Link"
-F 9 "/product-detail/en/texas-instruments/LP5907MFX-3.3-NOPB/296-38557-1-ND/5034443" H 10500 3250 60  0001 L CNN "DK_Detail_Page"
-F 10 "IC REG LINEAR 3.3V 250MA SOT23-5" H 10500 3350 60  0001 L CNN "Description"
-F 11 "Texas Instruments" H 10500 3450 60  0001 L CNN "Manufacturer"
-F 12 "Active" H 10500 3550 60  0001 L CNN "Status"
-	1    10300 2350
+P 10850 2350
+F 0 "U2" H 10850 2700 60  0000 C CNN
+F 1 "LP5907MFX-3_3_NOPB" H 10850 2800 60  0000 C CNN
+F 2 "Package_TO_SOT_SMD:SOT-23-5" H 11050 2550 60  0001 L CNN
+F 3 "http://www.ti.com/general/docs/suppproductinfo.tsp?distId=10&gotoUrl=http%3A%2F%2Fwww.ti.com%2Flit%2Fgpn%2Flp5907" H 11050 2650 60  0001 L CNN
+F 4 "296-38557-1-ND" H 11050 2750 60  0001 L CNN "Digi-Key_PN"
+F 5 "LP5907MFX-3.3/NOPB" H 11050 2850 60  0001 L CNN "MPN"
+F 6 "Integrated Circuits (ICs)" H 11050 2950 60  0001 L CNN "Category"
+F 7 "PMIC - Voltage Regulators - Linear" H 11050 3050 60  0001 L CNN "Family"
+F 8 "http://www.ti.com/general/docs/suppproductinfo.tsp?distId=10&gotoUrl=http%3A%2F%2Fwww.ti.com%2Flit%2Fgpn%2Flp5907" H 11050 3150 60  0001 L CNN "DK_Datasheet_Link"
+F 9 "/product-detail/en/texas-instruments/LP5907MFX-3.3-NOPB/296-38557-1-ND/5034443" H 11050 3250 60  0001 L CNN "DK_Detail_Page"
+F 10 "IC REG LINEAR 3.3V 250MA SOT23-5" H 11050 3350 60  0001 L CNN "Description"
+F 11 "Texas Instruments" H 11050 3450 60  0001 L CNN "Manufacturer"
+F 12 "Active" H 11050 3550 60  0001 L CNN "Status"
+	1    10850 2350
 	1    0    0    -1
 $EndComp
@@
 Text Label 12900 14450 0    50   ~ 0
 BL654_I2S_SD
+$Comp
+L Device:Fuse F1
+U 1 1 5E87E3DC
+P 10100 2150
+F 0 "F1" V 10180 2150 50  0000 C CNN
+F 1 "0603L075SLYR" V 10025 2150 50  0000 C CNN
+F 2 "Fuse:Fuse_0603_1608Metric" V 10030 2150 50  0001 C CNN
+F 3 "~" H 10100 2150 50  0001 C CNN
+F 4 "0603L075SLYR" V 10100 2150 50  0001 C CNN "MPN"
+	1    10100 2150
+	0    1    1    0
+$EndComp
+Wire Wire Line
+	9700 2150 9950 2150
+Wire Wire Line
+	10250 2150 10450 2150
+Connection ~ 10450 2150
+Text Label 6050 2200 0    50   ~ 0
+MCP73831_STAT
+Text Label 13950 6000 0    50   ~ 0
+MCP73831_STAT
+Text Label 13950 6200 0    50   ~ 0
+WS2812_DATA
+$Comp
+L LED:WS2812B D?
+U 1 1 5EA47254
+P 17150 4700
+F 0 "D?" H 17350 4925 50  0000 R BNN
+F 1 "WS2812B" H 17200 4475 50  0000 L TNN
+F 2 "APA-102-2020-256-8:LED_WS2812-2020" H 17200 4400 50  0001 L TNN
+F 3 "https://cdn-shop.adafruit.com/datasheets/WS2812B.pdf" H 17250 4325 50  0001 L TNN
+	1    17150 4700
+	1    0    0    -1
+$EndComp
+Text Label 16850 4700 2    50   ~ 0
+WS2812_DATA
+Text Label 17150 4250 0    50   ~ 0
+VIN
+Wire Wire Line
+	17150 4250 17150 4400
+$Comp
+L power:GND #PWR?
+U 1 1 5EA6E74F
+P 17150 5000
+F 0 "#PWR?" H 17150 4750 50  0001 C CNN
+F 1 "GND" H 17150 4850 50  0000 C CNN
+F 2 "" H 17150 5000 50  0001 C CNN
+F 3 "" H 17150 5000 50  0001 C CNN
+	1    17150 5000
+	1    0    0    -1
+$EndComp
 $EndSCHEMATC

Commit message: Changed layout and added button
Parts:
- added SW1: SW_Push, SW_B3U-3000P:SW_B3U-3000P, symbol Switch:SW_Push
- gave numbers to parts that had none: 1
Connections:
- net GND: now also SW1.2
- net at U1.6 (SIO_33): now also SW1.1
Changed lines of the file:
@@
 WS2812_DATA
 $Comp
-L LED:WS2812B D?
+L LED:WS2812B D2
 U 1 1 5EA47254
 P 17150 4700
-F 0 "D?" H 17350 4925 50  0000 R BNN
+F 0 "D2" H 17350 4925 50  0000 R BNN
 F 1 "WS2812B" H 17200 4475 50  0000 L TNN
 F 2 "APA-102-2020-256-8:LED_WS2812-2020" H 17200 4400 50  0001 L TNN
@@
 	17150 4250 17150 4400
 $Comp
-L power:GND #PWR?
+L power:GND #PWR022
 U 1 1 5EA6E74F
 P 17150 5000
-F 0 "#PWR?" H 17150 4750 50  0001 C CNN
+F 0 "#PWR022" H 17150 4750 50  0001 C CNN
 F 1 "GND" H 17150 4850 50  0000 C CNN
 F 2 "" H 17150 5000 50  0001 C CNN
@@
 	1    0    0    -1
 $EndComp
+$Comp
+L Switch:SW_Push SW1
+U 1 1 5E93ABDF
+P 15000 6500
+F 0 "SW1" H 15050 6600 50  0000 L CNN
+F 1 "SW_Push" H 15000 6440 50  0000 C CNN
+F 2 "SW_B3U-3000P:SW_B3U-3000P" H 15000 6700 50  0001 C CNN
+F 3 "~" H 15000 6700 50  0001 C CNN
+	1    15000 6500
+	1    0    0    -1
+$EndComp
+Wire Wire Line
+	14800 6500 13950 6500
+$Comp
+L power:GND #PWR023
+U 1 1 5E95EF4D
+P 15350 6750
+F 0 "#PWR023" H 15350 6500 50  0001 C CNN
+F 1 "GND" H 15350 6600 50  0000 C CNN
+F 2 "" H 15350 6750 50  0001 C CNN
+F 3 "" H 15350 6750 50  0001 C CNN
+	1    15350 6750
+	1    0    0    -1
+$EndComp
+Wire Wire Line
+	15350 6750 15350 6500
+Wire Wire Line
+	15350 6500 15200 6500
 $EndSCHEMATC

Commit message: Added board properties
Parts:
- removed J17, J18, J19, J20: 503480-0600, MOLEX_503480-0600:MOLEX_503480-0600, symbol 503480-0600:503480-0600
- removed J3: Conn_02x10_Odd_Even, DF23:DF23C-20DS-0.5V(51), symbol Connector_Generic:Conn_02x10_Odd_Even
Other:
- note added: "ACCELEROMETER"
- note added: "MICROPHONES"
- note added: "PPG SENSOR FPC"
- note added: "RGB LED"
- note added: "TEMP SENSOR FPC"
- moved on the sheet: C29, C30, J13, J14, MIC1, MIC2, R22, U5

Commit message: Main board routed
Connections:
- net +3V3: now also J4.1 (Pin_1)
- net ADS_CLK: now also U1.18 (SIO_15); no longer J11.8 (Pin_8), U1.30 (SIO_41), U3.17 (CLK)
- net ADS_SPI_MISO: now also U1.13 (SIO_20); no longer J11.3 (Pin_3), U1.51 (SIO_46/SPI_MISO), U3.21 (DOUT)
- net ADS_SPI_MOSI: now also U1.14 (SIO_19); no longer J11.4 (Pin_4), U1.56 (SIO_45/SPI_MOSI), U3.19 (DIN)
- net ADS_SPI_SCLK: now also U1.12 (SIO_21); no longer J11.2 (Pin_2), U1.53 (SIO_47/SPI_CLK), U3.20 (SCLK)
- net ADS_START: now also U1.21 (SIO_16); no longer J11.7 (Pin_7), U1.62 (SIO_42), U3.16 (START)
- net BL654_I2C_SCL_HV: no longer J13.2, U5.A2 (SCL)
- net BL654_I2C_SCL_LV: no longer J16.3, U6.2 (SCL)
- net BL654_I2C_SDA_HV: no longer J13.3, U5.A1 (SDA)
- net BL654_I2C_SDA_LV: no longer J16.4, U6.3 (SDA)
- net BL654_I2S_SCK: no longer J11.12 (Pin_12), MIC1.4 (BCLK), MIC2.4 (BCLK)
- net BL654_I2S_SD: no longer J11.13 (Pin_13), MIC1.6 (DATA_OUT), MIC2.6 (DATA_OUT), R22.1
- net BL654_I2S_WS: no longer J11.11 (Pin_11), MIC1.1 (WS), MIC2.1 (WS)
- net GND: now also C26.1
- net TMP_ADD0: now also U1.5 (SIO_35/NAUTORUN); no longer J13.5, U1.44 (SIO_31/AIN7), U5.C1 (ADD0)
- net TMP_ALERT: no longer J13.4, U5.C2 (ALERT)
- net VIN: now also C3.2, F1.1, U2.1 (IN), U2.3 (EN)
- net ~ADS_DRDY: now also U1.22 (SIO_14); no longer J11.9 (Pin_9), U1.32 (SIO_40), U3.22 (~DRDY)
- net ~ADS_PWDN_RESET: now also U1.16 (SIO_17); no longer J11.6 (Pin_6), U1.60 (SIO_43), U3.15 (~PWDN/RESET)
- net ~ADS_SPI_CS: now also U1.19 (NRESET/SIO_18); no longer J11.5 (Pin_5), U1.54 (SIO_44), U3.18 (~CS)
- net ~MAX_INT: now also U1.37 (SIO_07/UART_CTS); no longer J16.5, U6.13 (~INT)
- net VIN_FUSE: now reaches D3.K, F1.2, Q1.2 (S)
- net VIN_FUSE: no longer C3.2
- new net ADS_CLK_EXT: J11.8 (Pin_8), U3.17 (CLK)
- new net ADS_SPI_MISO_EXT: J11.3 (Pin_3), U3.21 (DOUT)
- new net ADS_SPI_MOSI_EXT: J11.4 (Pin_4), U3.19 (DIN)
- new net ADS_SPI_SCLK_EXT: J11.2 (Pin_2), U3.20 (SCLK)
- new net ADS_START_EXT: J11.7 (Pin_7), U3.16 (START)
- new net BL654_I2C_SCL_HV_EXT: J13.2, U5.A2 (SCL)
- new net BL654_I2C_SCL_LV_EXT: J16.3, U6.2 (SCL)
- new net BL654_I2C_SDA_HV_EXT: J13.3, U5.A1 (SDA)
- new net BL654_I2C_SDA_LV_EXT: J16.4, U6.3 (SDA)
- new net BL654_I2S_SCK_EXT: J11.12 (Pin_12), MIC1.4 (BCLK), MIC2.4 (BCLK)
- new net BL654_I2S_SD_EXT: J11.13 (Pin_13), MIC1.6 (DATA_OUT), MIC2.6 (DATA_OUT), R22.1
- new net BL654_I2S_WS_EXT: J11.11 (Pin_11), MIC1.1 (WS), MIC2.1 (WS)
- new net TMP_ADD0_EXT: J13.5, U5.C1 (ADD0)
- new net TMP_ALERT_EXT: J13.4, U5.C2 (ALERT)
- new net ~ADS_DRDY_EXT: J11.9 (Pin_9), U3.22 (~DRDY)
- new net ~ADS_PWDN_RESET_EXT: J11.6 (Pin_6), U3.15 (~PWDN/RESET)
- new net ~ADS_SPI_CS_EXT: J11.5 (Pin_5), U3.18 (~CS)
- new net ~MAX_INT_EXT: J16.5, U6.13 (~INT)
Other:
- moved on the sheet: C3, C4, F1, J11, J12, U2, U5

Commit message: Completed routing of all boards
Parts:
- removed J5, J6, J7, J8: 503480-0400, 503480-0400:MOLEX_503480-0400, symbol 503480-0400:503480-0400
- added J17, J3, J5, J8: 503480-0600, MOLEX_503480-0600:MOLEX_503480-0600, symbol 503480-0600:503480-0600
- added J18: ECG_RIGHT_LEG, MOLEX_503480-0600:ECG_SNAP, symbol Connector_Generic:Conn_01x01
- added J6: ECG_LEFT_ARM, MOLEX_503480-0600:ECG_SNAP, symbol Connector_Generic:Conn_01x01
- added J7: ECG_RIGHT_ARM, MOLEX_503480-0600:ECG_SNAP, symbol Connector_Generic:Conn_01x01
Connections:
- net +3V3: now also J17.6, J3.6, J5.1
- net BL654_I2S_SCK_EXT: now also J17.3, J3.3, J5.4, J8.4
- net BL654_I2S_SD_EXT: now also J17.2, J3.2, J5.5, J8.5
- net BL654_I2S_WS_EXT: now also J17.4, J3.4, J5.3, J8.3
- net GND: now also J10.S1 (SHIELD), J10.S2 (SHIELD), J9.S1 (SHIELD), J9.S2 (SHIELD), J17.1, J17.S1 (SHIELD), J17.S2 (SHIELD), J3.1, J3.S1 (SHIELD), J3.S2 (SHIELD), J5.6, J5.S1 (SHIELD), J5.S2 (SHIELD), J8.6, J8.S1 (SHIELD), J8.S2 (SHIELD)
- net LEFT_ARM renamed ECG_LEFT_ARM
- net ECG_LEFT_ARM: now also J3.5, J5.2, J6.1 (Pin_1)
- net RIGHT_ARM renamed ECG_RIGHT_ARM
- net ECG_RIGHT_ARM: now also J17.5, J7.1 (Pin_1), J8.2
- net RIGHT_LEG renamed ECG_RIGHT_LEG
- net ECG_RIGHT_LEG: now also J18.1 (Pin_1)
Other:
- moved on the sheet: J10, J9

Commit message: Fix temperature sensor thermal pad, mounting holes, silk screen, mic ground, capacitor symmetric location and routing
Parts:
- added J19: MOUNTING_HOLE_MAIN, MountingHole:MountingHole_2.2mm_M2_DIN965_Pad, symbol Connector_Generic:Conn_01x01
- added J20: MOUNTING_HOLE_ECG, MountingHole:MountingHole_2.2mm_M2_DIN965_Pad, symbol Connector_Generic:Conn_01x01
Connections:
- net GND: now also J19.1 (Pin_1), J20.1 (Pin_1)
- net MCP73831_STAT: now also U1.34 (SIO_04/AIN2); no longer U1.63 (SIO_38)
Changed lines of the file:
@@
 Wire Wire Line
 	5300 13550 5300 13700
-$Comp
-L power:GND #PWR0106
-U 1 1 5EAF82ED
-P 5450 15450
-F 0 "#PWR0106" H 5450 15200 50  0001 C CNN
-F 1 "GND" H 5450 15300 50  0000 C CNN
-F 2 "" H 5450 15450 50  0001 C CNN
-F 3 "" H 5450 15450 50  0001 C CNN
-	1    5450 15450
-	1    0    0    -1
-$EndComp
 Wire Wire Line
 	5450 15450 5450 15300
@@
 Text Label 6050 2200 0    50   ~ 0
 MCP73831_STAT
-Text Label 13950 6000 0    50   ~ 0
+Text Label 11550 6000 2    50   ~ 0
 MCP73831_STAT
 Text Label 13950 6200 0    50   ~ 0
@@
 Wire Wire Line
 	6450 12550 5500 12550
+$Comp
+L power:GND #PWR0106
+U 1 1 5EAF82ED
+P 5450 15450
+F 0 "#PWR0106" H 5450 15200 50  0001 C CNN
+F 1 "GND" H 5450 15300 50  0000 C CNN
+F 2 "" H 5450 15450 50  0001 C CNN
+F 3 "" H 5450 15450 50  0001 C CNN
+	1    5450 15450
+	1    0    0    -1
+$EndComp
+$Comp
+L Connector_Generic:Conn_01x01 J19
+U 1 1 5EAC4793
+P 19400 3700
+F 0 "J19" H 19400 3800 50  0000 C CNN
+F 1 "MOUNTING_HOLE_MAIN" V 19500 3700 50  0000 C CNN
+F 2 "MountingHole:MountingHole_2.2mm_M2_DIN965_Pad" H 19400 3700 50  0001 C CNN
+F 3 "~" H 19400 3700 50  0001 C CNN
+	1    19400 3700
+	0    -1   -1   0
+$EndComp
+$Comp
+L Connector_Generic:Conn_01x01 J20
+U 1 1 5EAC66C3
+P 20300 3700
+F 0 "J20" H 20300 3800 50  0000 C CNN
+F 1 "MOUNTING_HOLE_ECG" V 20400 3700 50  0000 C CNN
+F 2 "MountingHole:MountingHole_2.2mm_M2_DIN965_Pad" H 20300 3700 50  0001 C CNN
+F 3 "~" H 20300 3700 50  0001 C CNN
+	1    20300 3700
+	0    -1   -1   0
+$EndComp
+$Comp
+L power:GND #PWR0113
+U 1 1 5EAD18EB
+P 19400 3900
+F 0 "#PWR0113" H 19400 3650 50  0001 C CNN
+F 1 "GND" H 19400 3750 50  0000 C CNN
+F 2 "" H 19400 3900 50  0001 C CNN
+F 3 "" H 19400 3900 50  0001 C CNN
+	1    19400 3900
+	1    0    0    -1
+$EndComp
+$Comp
+L power:GND #PWR0114
+U 1 1 5EAD1E65
+P 20300 3900
+F 0 "#PWR0114" H 20300 3650 50  0001 C CNN
+F 1 "GND" H 20300 3750 50  0000 C CNN
+F 2 "" H 20300 3900 50  0001 C CNN
+F 3 "" H 20300 3900 50  0001 C CNN
+	1    20300 3900
+	1    0    0    -1
+$EndComp
 $EndSCHEMATC
