File: Lifedatalink_v1_revA.sch (KiCad schematic (older format))
At the start: 88 parts, among them J1 DX07S024XJ1R1100, J10 503480-0400, J11 5034801400, J12 5034801400, J13 503480-0600, J14 503480-0600, J15 503480-0600, J16 503480-0600, J17 503480-0600, J18 ECG_RIGHT_LEG, J19 MOUNTING_HOLE_MAIN, J2 BATTERY CONNECTOR, J20 MOUNTING_HOLE_ECG, J3 503480-0600, J4 Conn_01x06, J5 503480-0600, J6 ECG_LEFT_ARM, J7 ECG_RIGHT_ARM, J8 503480-0600, J9 503480-0400, Q1 DMG2301L, SW1 SW_Push, U1 BL654, U2 LP5907MFX-3_3_NOPB, U3 ADS1292R, U4 MCP73831-2-OT, U5 TMP117NAIYBGR, U6 MAX30102, U7 LP5907MFX-1.8, U8 IIS2DLPCTR, U9 PCA9306, Y1 Crystal

Commit message: Finished post routing schematic pinout and footprint cross check
Parts:
- added C31: 100pF, Capacitor_SMD:C_0402_1005Metric, symbol Device:C
- D1: footprint digikey-footprints:UFDFN-6_1.45x1mm -> SnapEda:SON50P100X145X60-6N
- D2: MPN (none) -> APA-102-2020
- D3: footprint Diode_SMD:D_SOD-123F -> Diode_SMD:D_SOD-123
- F1: value 0603L075SLYR -> 0ZCK0075FF2E; footprint Fuse:Fuse_0603_1608Metric -> Fuse:Fuse_0805_2012Metric
- J1: MPN (none) -> DX07S024XJ1R1100
- J10, J9: MPN (none) -> 503480-0400
- J11, J12: MPN (none) -> 503480-1400
- J13, J14, J15, J16, J17, J3, J5, J8: MPN (none) -> 503480-0600
- J2: value BATTERY CONNECTOR -> SM02B-SRSS-TB(LF)(SN); footprint Connector_JST:JST_SH_BM02B-SRSS-TB_1x02-1MP_P1.00mm_Vertical -> Connector_JST:JST_SH_SM02B-SRSS-TB_1x02-1MP_P1.00mm_Horizontal; MPN (none) -> SM02B-SRSS-TB(LF)(SN)
- Q1: value DMG2301L -> CSD23280F3; footprint Package_TO_SOT_SMD:SOT-23 -> SnapEda:TRANS_CSD23280F3; MPN (none) -> CSD23280F3
- SW1: MPN (none) -> B3U-3000P
- U1: MPN (none) -> BL654
- U3: MPN (none) -> ADS1292R
- U4: MPN (none) -> MCP73831-2-OT
- U5: MPN (none) -> TMP117NAIYBGR
- U7: MPN (none) -> LP5907MFX-1.8
- U8: MPN (none) -> IIS2DLPCTR
- U9: MPN (none) -> PCA9306
Connections:
- net +1V8: now also R18.1, R19.1, U9.2 (VREF1); no longer R17.1, R20.1, R21.1, U9.7 (VREF2)
- net +3V3: now also J13.6, J17.1, J8.6, R17.1, R20.1, R21.1, U9.7 (VREF2); no longer J13.1, J17.6, R18.1, R19.1, U9.2 (VREF1)
- net BL654_I2C_SCL_HV: now also R20.2, U9.6 (SCL2); no longer R19.2, U9.3 (SCL1)
- net BL654_I2C_SCL_HV_EXT: now also J13.5; no longer J13.2
- net BL654_I2C_SCL_LV: now also R19.2, U9.3 (SCL1); no longer R20.2, U9.6 (SCL2)
- net BL654_I2C_SDA_HV: now also R21.2, U9.5 (SDA2); no longer R18.2, U9.4 (SDA1)
- net BL654_I2C_SDA_HV_EXT: now also J13.4; no longer J13.3
- net BL654_I2C_SDA_LV: now also R18.2, U9.4 (SDA1); no longer R21.2, U9.5 (SDA2)
- net BL654_I2S_SCK_EXT: now also J17.4, J8.3; no longer J17.3, J8.4
- net BL654_I2S_SD_EXT: now also J17.5, J8.2; no longer J17.2, J8.5
- net BL654_I2S_WS_EXT: now also J17.3, J8.4; no longer J17.4, J8.3
- net ECG_RIGHT_ARM: now also J17.2, J8.5; no longer J17.5, J8.2
- net ECG_RIGHT_LEG: now also J10.4; no longer J10.1
- net GND: now also J10.1, J13.1, J17.6, J8.1, J9.4, C31.1; no longer J13.6, J17.1, J8.6
- net TMP_ADD0_EXT: now also J13.2; no longer J13.5
- net TMP_ALERT_EXT: now also J13.3; no longer J13.4
- net at R17.2, U9.8 (EN): now also C31.2
Other:
- moved on the sheet: J17, J18, J8

Commit message: Added battery level voltage divider
Parts:
- added R1, R2: 100K, Resistor_SMD:R_0402_1005Metric, symbol Device:R
Connections:
- net +BATT: now also R1.2
- net GND: now also R2.1
- net VDIV: now reaches U1.48 (SIO_29/AIN5)
- net VDIV: now also R1.1, R2.2
Changed lines of the file:
@@
 	19600 12500 19600 12750
 $Comp
-L power:GND #PWR?
+L power:GND #PWR097
 U 1 1 5EBDDE80
 P 19850 12800
-F 0 "#PWR?" H 19850 12550 50  0001 C CNN
+F 0 "#PWR097" H 19850 12550 50  0001 C CNN
 F 1 "GND" H 19850 12650 50  0000 C CNN
 F 2 "" H 19850 12800 50  0001 C CNN
@@
 Wire Wire Line
 	19600 12500 19950 12500
+Text Label 13950 7000 0    50   ~ 0
+VDIV
+$Comp
+L power:+BATT #PWR095
+U 1 1 5EA0807E
+P 9550 3400
+F 0 "#PWR095" H 9550 3250 50  0001 C CNN
+F 1 "+BATT" H 9550 3540 50  0000 C CNN
+F 2 "" H 9550 3400 50  0001 C CNN
+F 3 "" H 9550 3400 50  0001 C CNN
+	1    9550 3400
+	1    0    0    -1
+$EndComp
+$Comp
+L Device:R R1
+U 1 1 5EA08810
+P 9550 3550
+F 0 "R1" V 9630 3550 50  0000 C CNN
+F 1 "100K" V 9550 3550 50  0000 C CNN
+F 2 "Resistor_SMD:R_0402_1005Metric" V 9480 3550 50  0001 C CNN
+F 3 "~" H 9550 3550 50  0001 C CNN
+	1    9550 3550
+	-1   0    0    1
+$EndComp
+$Comp
+L Device:R R2
+U 1 1 5EA091FA
+P 9550 3950
+F 0 "R2" V 9630 3950 50  0000 C CNN
+F 1 "100K" V 9550 3950 50  0000 C CNN
+F 2 "Resistor_SMD:R_0402_1005Metric" V 9480 3950 50  0001 C CNN
+F 3 "~" H 9550 3950 50  0001 C CNN
+	1    9550 3950
+	-1   0    0    1
+$EndComp
+$Comp
+L power:GND #PWR096
+U 1 1 5EA09827
+P 9550 4100
+F 0 "#PWR096" H 9550 3850 50  0001 C CNN
+F 1 "GND" H 9550 3950 50  0000 C CNN
+F 2 "" H 9550 4100 50  0001 C CNN
+F 3 "" H 9550 4100 50  0001 C CNN
+	1    9550 4100
+	1    0    0    -1
+$EndComp
+Wire Wire Line
+	9550 3700 9550 3750
+Text Label 9850 3750 0    50   ~ 0
+VDIV
+Wire Wire Line
+	9850 3750 9550 3750
+Connection ~ 9550 3750
+Wire Wire Line
+	9550 3750 9550 3800
 $EndSCHEMATC

Commit message: Fixed electrode boards
Connections:
- net ECG_RIGHT_LEG: now also J10.1; no longer J10.4
- net GND: now also J10.4; no longer J10.1
Other:
- moved on the sheet: J18
Changed lines of the file:
@@
 Text Label 7550 6750 0    50   ~ 0
 ECG_RIGHT_ARM
-Text Label 5500 12850 0    50   ~ 0
+Text Label 5500 12550 0    50   ~ 0
 ECG_RIGHT_LEG
 Text Label 3500 12550 2    50   ~ 0
@@
 L Connector_Generic:Conn_01x01 J18
 U 1 1 5E9073B1
-P 6650 12850
-F 0 "J18" H 6650 12950 50  0000 C CNN
-F 1 "ECG_RIGHT_LEG" H 6650 12750 50  0000 C CNN
-F 2 "MOLEX_503480-0600:ECG_SNAP" H 6650 12850 50  0001 C CNN
-F 3 "~" H 6650 12850 50  0001 C CNN
-	1    6650 12850
-	1    0    0    -1
-$EndComp
-Wire Wire Line
-	6450 12850 5500 12850
+P 6650 12550
+F 0 "J18" H 6650 12650 50  0000 C CNN
+F 1 "ECG_RIGHT_LEG" H 6650 12450 50  0000 C CNN
+F 2 "MOLEX_503480-0600:ECG_SNAP" H 6650 12550 50  0001 C CNN
+F 3 "~" H 6650 12550 50  0001 C CNN
+	1    6650 12550
+	1    0    0    -1
+$EndComp
+Wire Wire Line
+	6450 12550 5500 12550
 $Comp
 L power:GND #PWR0106
@@
 	-1   0    0    -1
 $EndComp
-Wire Wire Line
-	3500 12850 3400 12850
-Wire Wire Line
-	3400 12850 3400 13050
-Connection ~ 3400 13050
-$Comp
-L power:GND #PWR0116
-U 1 1 5EE4B4E9
-P 5500 12550
-F 0 "#PWR0116" H 5500 12300 50  0001 C CNN
-F 1 "GND" H 5500 12400 50  0000 C CNN
-F 2 "" H 5500 12550 50  0001 C CNN
-F 3 "" H 5500 12550 50  0001 C CNN
-	1    5500 12550
-	1    0    0    1
-$EndComp
 $Comp
 L Lifedatalink_v1_revA-rescue:+3.3V-power #PWR065
@@
 Wire Wire Line
 	9550 3750 9550 3800
+Wire Wire Line
+	3500 12850 3400 12850
+Connection ~ 3400 13050
+Wire Wire Line
+	3400 12850 3400 13050
+Wire Wire Line
+	5500 12850 5600 12850
+Wire Wire Line
+	5600 12850 5600 13050
+Connection ~ 5600 13050
 $EndSCHEMATC

Commit message: Finalized and exported CAD files for quotation
Parts:
- C1: MPN (none) -> C0402C120J5GACTU
- C10, C17, C19, C23, C27, C8: MPN (none) -> C0402C104K4PACTU
- C11, C12, C24, C25, C26, C3, C4: MPN (none) -> C0402C105K9PACTU
- C13, C14: MPN (none) -> C0402C473K3RACAUTO
- C15, C16, C18, C20: MPN (none) -> C0402C222K5RACTU
- C2: MPN (none) -> C0402C100J5GACTU
- C21: MPN (none) -> C0402C470K5GACTU
- C22, C28, C5, C9: MPN (none) -> C0402C106M9PAC7867
- C29, C30: value 0.1uF -> 100nF; MPN (none) -> C0402C104K4PACTU
- C31: MPN (none) -> C0402C101J5GACTU
- C6, C7: MPN (none) -> C0402C475M7PACTU
- R1, R12, R14, R2, R22, R4: MPN (none) -> CRCW0402100KFKEDC
- R10, R5, R6, R9: MPN (none) -> CRCW040210M0FKED
- R11: MPN (none) -> CRCW04021M00FKEDC
- R13: MPN (none) -> CRCW04020000Z0EDC
- R15, R16: MPN (none) -> RC0402FR-0745K3L
- R17: MPN (none) -> RC0402FR-07200KL
- R18, R19, R20, R21: MPN (none) -> CRCW04024K70FKEDC
- R3: MPN (none) -> CRCW040210K0FKEDC
- R7, R8: MPN (none) -> CRCW040240K2FKEDC
- U3: value ADS1292R -> ADS1292RIRSMT; MPN ADS1292R -> ADS1292RIRSMT
- U4: value MCP73831-2-OT -> MCP73831T-2ACI/OT; MPN MCP73831-2-OT -> MCP73831T-2ACI/OT
- U7: value LP5907MFX-1.8 -> LP5907MFX-1.8/NOPB; MPN LP5907MFX-1.8 -> LP5907MFX-1.8/NOPB
- U9: value PCA9306 -> PCA9306DQER; MPN PCA9306 -> PCA9306DQER
